File: fpgaler.kicad_pcb (KiCad board)
At the start: 4 copper layers, 100 x 100 mm, 297 parts, among them J1 USB_C_Receptacle_USB2.0, J3 JTAG, J4 FTDI_RST, J5 VGA, J6 DB9 Expander 1, J7 DB9 Expander 0, Q1 BC817, SW1 ROT, SW2 ROT1, SW3 K1, SW4 K2, SW5 PROGRAM, SW6 K3, SW7 FPGA GSRN, SW8 K4, U1 TLV62569DRL, U10 XC6206PxxxMR, U11 IS62WV51216BLL-55TLI, U2 TLV62569DRL, U3 NCP115-2.5, U5 93LC56BT-I/OT, U6 FT2232HL, U7 CAT24C128, U8 LFE5U-25F-8MG285C, U9 W25Q128JVP, X1 27MHz, Y1 7M-12.000MAAJ

Commit message: Plase silkscreen
Parts:
- added D14: 1.1V, Diode_SMD:D_0603_1608Metric, F.Cu at (168.0, 84.5)
- added D15: logo, Diode_SMD:D_0603_1608Metric, F.Cu at (151.5, 76.5)
- added G***: LOGO, kicad:fvga2, F.Cu at (163.4, 74.1)
- added Q2: BC817, Package_TO_SOT_SMD:SOT-23, F.Cu at (169.0, 102.8)
- added R36: 1.2k, Resistor_SMD:R_0603_1608Metric, F.Cu at (164.8, 100.7)
- added R37: 1.2k, Resistor_SMD:R_0603_1608Metric, F.Cu at (164.8, 103.2)
- added R38: 1.2k, Resistor_SMD:R_0603_1608Metric, F.Cu at (146.8, 78.5)
- added TP37: GND, TestPoint:TestPoint_THTPad_D1.5mm_Drill0.7mm, F.Cu at (176.3, 65.1)
- added TP38: 5V, TestPoint:TestPoint_THTPad_D1.5mm_Drill0.7mm, F.Cu at (172.8, 103.0)
- added TP39: TestPoint, TestPoint:TestPoint_THTPad_D1.5mm_Drill0.7mm, F.Cu at (146.8, 75.5)
- TP27: value TestPoint -> 3.3V
- TP35: value TestPoint -> 2.5V
- TP36: value TestPoint -> 5V
- moved TP36 50.8 mm to (157.1, 66.1)
- moved R35 50.3 mm to (157.1, 69.1), turned to -90 degrees
- moved D10 48.2 mm to (171.0, 70.5), turned to 86 degrees
- moved D13 48.1 mm to (163.4, 69.7), turned to -178 degrees
- moved R25 44.2 mm to (152.8, 84.0), turned to -90 degrees
- moved TP27 43.7 mm to (152.8, 80.8)
- moved TP35 43.7 mm to (176.4, 71.6)
- moved R26 41.4 mm to (176.4, 74.7), turned to -90 degrees
- moved D9 38.2 mm to (163.8, 84.5)
- moved R105 28.4 mm to (139.0, 78.5), turned to 0 degrees
- moved R106 26.2 mm to (139.0, 76.8), turned to 0 degrees
- moved R107 24.1 mm to (139.0, 75.0), turned to 0 degrees
- moved R108 21.8 mm to (139.0, 73.1), turned to 0 degrees
- moved R109 19.8 mm to (139.0, 71.3), turned to 0 degrees
- moved R110 18.0 mm to (139.0, 69.5), turned to 0 degrees
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Connections:
- U8 pad A15: unconnected-(U8F-PL14D-PadA15) -> /FPGA/Led_log
Routing:
- net /FPGA/VGA_B0: track 45.6 -> 15.6 mm
- net /FPGA/VGA_B1: track 43.2 -> 16.8 mm
- net /FPGA/VGA_B2: track 41.5 -> 18.1 mm
- net /FPGA/VGA_G0: track 40.8 -> 21.4 mm
- net /FPGA/VGA_G1: track 38.9 -> 22.7 mm
- net /FPGA/VGA_G2: track 36.5 -> 24.2 mm
- net /B: track 14.5 -> 26.6 mm
- net /G: track 11.9 -> 22.8 mm
- net /FPGA/VGA_R0: track 35.6 -> 26.9 mm
- net /R: track 10.5 -> 18.2 mm
- net /FPGA/VGA_VSYNC: track 28.4 -> 35.1 mm
- net /FPGA/VGA_R1: track 33.3 -> 28.2 mm
- net /FPGA/VGA_HSYNC: track 30.0 -> 33.3 mm
- net /FPGA/VGA_R2: track 32.3 -> 30.5 mm
- net /HSYNC: track 22.3 -> 24.1 mm
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Other:
- board text added: "FVGA"
