File: fpga_pwr.kicad_sch (KiCad schematic)
At the start: 29 parts, among them Q1 BC817, U8 LFE5U-25F-8MG285C

Commit message: Place planes
Changed lines of the file:
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@@
+		)
+	)
+	(global_label "SPI_CONFIG_SCK"
+		(shape input)
+		(at 189.23 52.07 0)
+		(effects
+			(font
+				(size 1.27 1.27)
+			)
+			(justify left)
+		)
+		(property "Intersheetrefs" "${INTERSHEET_REFS}"
+			(at 189.23 52.07 0)
+			(effects
+				(font
+					(size 1.27 1.27)
+				)
+				(hide yes)
+			)
 		)
 	)
@@
 		(effects
 			(font
-				(size 1.27 1.27)
-			)
-			(justify left)
-		)
-	)
-	(hierarchical_label "SPI_CONFIG_SCK"
-		(shape input)
-		(at 189.23 52.07 0)
-		(effects
-			(font
