File: fpgaler.kicad_sch (KiCad schematic)
At the start: 99 parts, among them J1 USB_C_Receptacle_USB2.0, J3 JTAG, J4 FTDI_RST, J5 VGA, J6 DB9 Expander, J7 DB9 Expander, SW1 RotaryEncoder_Switch, SW2 RotaryEncoder_Switch, SW3 K1, SW4 K2, SW5 PROGRAMN, SW6 K3, SW7 FPGA GSRN, SW8 K4

Commit message: Place planes
Parts:
- added FB7: 15Ω@100MHz, Inductor_SMD:L_0603_1608Metric_Pad1.05x0.95mm_HandSolder, symbol Device:FerriteBead
Connections:
- net GND: now also FB7.2; no longer J1.A1 (GND), J1.A12 (GND), J1.B1 (GND), J1.B12 (GND), J1.S1 (SHIELD)
- new net: FB7.1, J1.A1 (GND), J1.A12 (GND), J1.B1 (GND), J1.B12 (GND), J1.S1 (SHIELD)
- no-connect marks 55 -> 54
Other:
- sheet FPGA PWR ports: added none; removed SPI_CONFIG_SCK
Changed lines of the file:
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@@
 	)
 	(no_connect
-		(at 201.93 33.02)
-	)
-	(no_connect
 		(at 110.49 105.41)
 	)
@@
 	(wire
 		(pts
-			(xy 26.67 77.47) (xy 26.67 81.28)
-		)
-		(stroke
-			(width 0)
-			(type default)
-		)
-	)
-	(wire
-		(pts
 			(xy 146.05 165.1) (xy 146.05 170.18)
 		)
@@
 	(wire
 		(pts
+			(xy 26.67 77.47) (xy 26.67 86.36)
+		)
+		(stroke
+			(width 0)
+			(type default)
+		)
+	)
+	(wire
+		(pts
 			(xy 180.34 40.64) (xy 157.48 40.64)
 		)
@@
 	(wire
 		(pts
+			(xy 36.83 86.36) (xy 26.67 86.36)
+		)
+		(stroke
+			(width 0)
+			(type default)
+		)
+	)
+	(wire
+		(pts
 			(xy 234.95 101.6) (xy 241.3 101.6)
 		)
@@
 	)
 	(symbol
+		(lib_id "Device:FerriteBead")
+		(at 40.64 86.36 90)
+		(unit 1)
+		(exclude_from_sim no)
+		(in_bom yes)
+		(on_board yes)
+		(dnp no)
+		(fields_autoplaced yes)
+		(property "Reference" "FB7"
+			(at 40.5892 78.74 90)
+			(effects
+				(font
+					(size 1.27 1.27)
+				)
+			)
+		)
+		(property "Value" "15Ω@100MHz"
+			(at 40.5892 81.28 90)
+			(effects
+				(font
+					(size 1.27 1.27)
+				)
+			)
+		)
+		(property "Footprint" "Inductor_SMD:L_0603_1608Metric_Pad1.05x0.95mm_HandSolder"
+			(at 40.64 88.138 90)
+			(effects
+				(font
+					(size 1.27 1.27)
+				)
+				(hide yes)
+			)
+		)
+		(property "Datasheet" "~"
+			(at 40.64 86.36 0)
+			(effects
+				(font
+					(size 1.27 1.27)
+				)
+				(hide yes)
+			)
+		)
+		(property "Description" "CBG160808U150T"
+			(at 40.64 86.36 0)
+			(effects
+				(font
+					(size 1.27 1.27)
+				)
+				(hide yes)
+			)
+		)
+		(property "KLC_S3.3" ""
+			(at 40.64 86.36 90)
+			(effects
+				(font
+					(size 1.27 1.27)
+				)
+				(hide yes)
+			)
+		)
+		(property "KLC_S4.1" ""
+			(at 40.64 86.36 90)
+			(effects
+				(font
+					(size 1.27 1.27)
+				)
+				(hide yes)
+			)
+		)
+		(pin "1"
+		)
+		(pin "2"
+		)
+		(instances
+			(project "fpgaler"
+				(path "/d6c42660-1080-4fbd-a2d9-2a0cd6b4e770"
+					(reference "FB7")
+					(unit 1)
+				)
+			)
+		)
+	)
+	(symbol
 		(lib_id "power:GND")
 		(at 137.16 187.96 0)
@@
 	(symbol
 		(lib_id "power:GND")
-		(at 26.67 81.28 0)
+		(at 44.45 86.36 0)
 		(unit 1)
 		(exclude_from_sim no)
@@
 		(fields_autoplaced yes)
 		(property "Reference" "#PWR03"
-			(at 26.67 87.63 0)
+			(at 44.45 92.71 0)
 			(effects
 				(font
@@
 		)
 		(property "Value" "GND"
-			(at 26.67 86.36 0)
+			(at 46.99 87.6299 0)
 			(effects
 				(font
 					(size 1.27 1.27)
 				)
+				(justify left)
 			)
 		)
 		(property "Footprint" ""
-			(at 26.67 81.28 0)
+			(at 44.45 86.36 0)
 			(effects
 				(font
@@
 		)
 		(property "Datasheet" ""
-			(at 26.67 81.28 0)
+			(at 44.45 86.36 0)
 			(effects
 				(font
@@
 		)
 		(property "Description" "Power symbol creates a global label with name \"GND\" , ground"
-			(at 26.67 81.28 0)
+			(at 44.45 86.36 0)
 			(effects
 				(font
@@
 			)
 		)
-		(pin "SPI_CONFIG_SCK" input
-			(at 201.93 33.02 0)
-			(effects
-				(font
-					(size 1.27 1.27)
-				)
-				(justify right)
-			)
-		)
