File: fpgaler.kicad_sch (KiCad schematic)
At the start: 109 parts, among them J1 USB_C_Receptacle_USB2.0, J3 JTAG, J4 FTDI_RST, J5 VGA, J6 DB9 Expander 1, J7 DB9 Expander 0, SW1 ROT, SW2 ROT1, SW3 K1, SW4 K2, SW5 PROGRAM, SW6 K3, SW7 FPGA GSRN, SW8 K4

Commit message: Plase silkscreen
Parts:
- added D14: 1.1V, Diode_SMD:D_0603_1608Metric, symbol Device:LED
- added D15: logo, Diode_SMD:D_0603_1608Metric, symbol Device:LED
- added Q2: BC817, Package_TO_SOT_SMD:SOT-23, symbol Transistor_BJT:BC817
- added R36, R37, R38: 1.2k, Resistor_SMD:R_0603_1608Metric, symbol Device:R
- added TP37: GND, TestPoint:TestPoint_THTPad_D1.5mm_Drill0.7mm, symbol Connector:TestPoint
- added TP38: 5V, TestPoint:TestPoint_THTPad_D1.5mm_Drill0.7mm, symbol Connector:TestPoint
- added TP39: TestPoint, TestPoint:TestPoint_THTPad_D1.5mm_Drill0.7mm, symbol Connector:TestPoint
- TP27: value TestPoint -> 3.3V
- TP35: value TestPoint -> 2.5V
- TP36: value TestPoint -> 5V
Connections:
- net +3.3V: now also R36.2
- net GND: now also D15.1 (K), Q2.2 (E), TP37.1
- new net: D14.1 (K), Q2.3 (C)
- new net: D14.2 (A), R36.1
- new net: D15.2 (A), R38.2
- new net: Q2.1 (B), R37.1
- new net +1.1V: R37.2, TP38.1
- new net FPGA/Led_log: R38.1, TP39.1
Other:
- sheet FPGA ports: added Led_log; removed none
- moved on the sheet: C7, D10, D13, D9, J3, R22, R25, R26, R35, SW7, TP27, TP35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

Commit message: Start to fix dcr
Parts:
- TP38: value 5V -> 1.1V
Changed lines of the file:
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@@
 			)
 		)
-		(property "Value" "5V"
+		(property "Value" "1.1V"
 			(at 113.03 109.982 90)
 			(effects
