File: FPGA.kicad_sch (KiCad schematic)
At the start: 91 parts, among them U11 IS62WV51216BLL-55TLI, U7 CAT24C128, U8 LFE5U-25F-8MG285C, U9 W25Q128JVP, X1 27MHz

Commit message: Plase silkscreen
Connections:
- net Led_log: now reaches U8.A15 (PL14D)
- no-connect marks 95 -> 94
Changed lines of the file:
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@@
 	)
 	(no_connect
-		(at 229.87 128.27)
-	)
-	(no_connect
 		(at 224.79 33.02)
 	)
@@
 	(wire
 		(pts
+			(xy 229.87 128.27) (xy 260.35 128.27)
+		)
+		(stroke
+			(width 0)
+			(type default)
+		)
+	)
+	(wire
+		(pts
 			(xy 270.51 83.82) (xy 260.35 83.82)
 		)
@@
 		(effects
 			(font
+				(size 1.27 1.27)
+			)
+			(justify left)
+		)
+	)
+	(hierarchical_label "Led_log"
+		(shape input)
+		(at 260.35 128.27 0)
+		(effects
+			(font
